File: dod-250-clone.kicad_sch (KiCad schematic)
At the start: 36 parts, among them U1 LM741

Commit message: Fix silkscreen for wire holes
Parts:
- H10: value SW_OUT -> OUT
- H11: value SW_GND -> GND
- H12: value SW_LED -> LED
- H5: value SW_IN -> IN
- H6: value SW_SEND -> SEND
- H7: value SW_RTN -> RTN
Changed lines of the file:
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@@
 			)
 		)
-		(property "Value" "SW_GND"
+		(property "Value" "GND"
 			(at 78.74 168.9099 0)
 			(effects
@@
 			)
 		)
-		(property "Value" "SW_LED"
+		(property "Value" "LED"
 			(at 115.57 168.9099 0)
 			(effects
@@
 			)
 		)
-		(property "Value" "SW_OUT"
+		(property "Value" "OUT"
 			(at 135.89 160.0199 0)
 			(effects
@@
 			)
 		)
-		(property "Value" "SW_SEND"
+		(property "Value" "SEND"
 			(at 78.74 160.0199 0)
 			(effects
@@
 			)
 		)
-		(property "Value" "SW_IN"
+		(property "Value" "IN"
 			(at 57.15 160.0199 0)
 			(effects
@@
 			)
 		)
-		(property "Value" "SW_RTN"
+		(property "Value" "RTN"
 			(at 115.57 160.0199 0)
 			(effects

Commit message: Fix pot footprints
Parts:
- RV1, RV2: footprint Potentiometer_THT:Potentiometer_Omeg_PC16BU_Vertical -> Floodlight_Custom_Footprints:Alpha_RV16AF-41
Changed lines of the file:
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@@
 			)
 		)
-		(property "Footprint" "Potentiometer_THT:Potentiometer_Omeg_PC16BU_Vertical"
+		(property "Footprint" "Floodlight_Custom_Footprints:Alpha_RV16AF-41"
 			(at 92.71 93.98 0)
 			(effects
@@
 			)
 		)
-		(property "Footprint" "Potentiometer_THT:Potentiometer_Omeg_PC16BU_Vertical"
+		(property "Footprint" "Floodlight_Custom_Footprints:Alpha_RV16AF-41"
 			(at 236.22 118.11 0)
 			(effects
